File: gerbalino0.3.1.brd (EAGLE design)
At the start: 47 parts, among them IC1 7805TV, Q1 16mhz

Commit message: gerbalino bug fixes v0.3.1
Parts:
- removed R3: 0, 01_SparkFun:1206
- R7: value 499 -> 1k
- moved R2 28.9 mm to (86.7, 54.0), turned to 180 degrees
- moved R6 4.83 mm to (15.7, 35.6), turned to 0 degrees
- moved R8 4.64 mm to (15.7, 44.8), turned to 0 degrees
- moved C1 4.18 mm to (44.9, 32.6), turned to 90 degrees
- moved R9 3.24 mm to (85.3, 40.1)
- moved U$7 2.92 mm to (79.1, 40.1), turned to 180 degrees
- moved DC_MOTOR 2.73 mm to (49.5, 54.2)
- moved ENDSTOP_X 2.73 mm to (75.8, 54.2)
- moved ENDSTOP_Y 2.73 mm to (68.6, 54.2)
- moved ENDSTOP_Z 2.73 mm to (61.4, 54.2)
- moved ENDSTOP_Z1 2.73 mm to (30.7, 54.4)
- moved ENDSTOP_Z2 2.73 mm to (20.1, 54.2)
- moved ENDSTOP_Z3 2.73 mm to (37.8, 54.4)
- moved C7 2.41 mm to (7.37, 24.6)
- moved ENDSTOP_Z4 2.35 mm to (3.94, 54.2)
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Connections:
- removed net N$40: R3.2, U$1.STEP
- removed net N$8: R8.2, U$6.2
- new net N$25: R6.2, U$5.1
- net +5V: now also R6.1, R8.1, R9.1
- net ENABLE: now also U$7.2; no longer U$7.1
- net GND: no longer R6.1, R8.1, R9.1
- net N$23: now also U$7.1; no longer U$7.2
- net N$7: now also R8.2, U$6.1; no longer R6.2, U$5.2
- net RX: now also U$6.2; no longer U$6.1
- net STEP_Y: now also U$1.STEP; no longer R3.1
- net TX: now also U$5.2; no longer U$5.1
Routing:
- net GND: track 466.0 -> 433.6 mm
- net N$40: track 21.0 -> 0.00 mm
- net +5V: track 272.7 -> 291.8 mm
- net STEP_Y: track 10.3 -> 17.9 mm
- net STEP_X: track 37.5 -> 29.9 mm
- net N$8: track 4.14 -> 0.00 mm
- net N$1: track 6.65 -> 2.60 mm
- net DIR_X: track 76.4 -> 79.2 mm
- net LIMIT_X: track 40.9 -> 43.7 mm
- net SCK: track 5.35 -> 8.08 mm
- net PROBE: track 24.5 -> 27.2 mm
- net MOSI: track 9.53 -> 12.3 mm
- net GRBL_RESET: track 8.88 -> 11.6 mm
- net COOL: track 16.4 -> 19.2 mm
- net LIMIT_Y: track 33.0 -> 35.7 mm
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Other:
- board text added: "GeRBaLINO V0.3.1"
- board text removed: "GeRBaLINO V0.3"
