File: gerbalino0.3.1.sch (EAGLE design)
At the start: 47 parts, among them IC1 7805TV, Q1 16mhz

Commit message: gerbalino bug fixes v0.3.1
Parts:
- removed R3: 0, 01_SparkFun:RESISTOR1206
- R7: value 499 -> 1k
Connections:
- removed net N$40: R3.2, U$1.STEP
- removed net N$8: R8.2, U$6.C
- new net N$25: R6.2, U$5.A
- net +5V: now also R6.1, R8.1, R9.1
- net ENABLE: now also U$7.C; no longer U$7.A
- net GND: no longer R6.1, R8.1, R9.1
- net N$23: now also U$7.A; no longer U$7.C
- net N$7: now also R8.2, U$6.A; no longer R6.2, U$5.C
- net RX: now also U$6.C; no longer U$6.A
- net STEP_Y: now also U$1.STEP; no longer R3.1
- net TX: now also U$5.C; no longer U$5.A
Other:
- moved on the sheet: R2, U$5, U$6, U$7
